File: yuho.kicad_pcb (KiCad board)
At the start: 2 copper layers, 70 x 164.1 mm, 137 parts, among them J1 Conn_02x05_Odd_Even, J2 Conn_02x04_Odd_Even, J3 47219-2001, J4 Conn_02x04_Odd_Even, Q1 2N7002K, Q10 2N7002K, Q11 SSM3K344R, Q2 ST-1KL3A, Q3 2N7002K, Q4 ST-1KL3A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

Commit message: 発注用のもの(だと信じたい)ver
Parts:
- removed Q11: SSM3K344R, Fusoku:2SC2712GRLF
- added C27: 0.1μ, Capacitor_SMD:C_0603_1608Metric_Pad1.08x0.95mm_HandSolder, F.Cu at (98.0, 126.7)
- added Q12: AO3400A, Package_TO_SOT_SMD:SOT-23, F.Cu at (89.7, 145.8)
- C1: value 10μ -> 22μ; footprint Capacitor_SMD:C_0603_1608Metric_Pad1.08x0.95mm_HandSolder -> Capacitor_SMD:C_1210_3225Metric_Pad1.33x2.70mm_HandSolder
- C2: value 0.1μ -> 1.0μ
- C3: footprint Capacitor_SMD:C_0603_1608Metric_Pad1.08x0.95mm_HandSolder -> Capacitor_SMD:C_0805_2012Metric_Pad1.18x1.45mm_HandSolder
- C4: value 2.2μ -> 4.7μ; footprint Capacitor_SMD:C_0603_1608Metric_Pad1.08x0.95mm_HandSolder -> Capacitor_SMD:C_0805_2012Metric_Pad1.18x1.45mm_HandSolder
- Q9: value IRLML6402 -> AO3407A
- R11, R3, R5, R8: value 10 -> 20
- moved R19 115.8 mm to (153.4, 100.6), turned to -90 degrees
- moved SW4 114.4 mm to (150.6, 97.4), turned to -90 degrees
- moved SW3 112.6 mm to (146.2, 92.6), turned to 180 degrees
- moved D14 109.4 mm to (148.9, 101.8), turned to 180 degrees
- moved D15 108.4 mm to (148.9, 103.3), turned to 180 degrees
- moved R28 108.3 mm to (153.8, 116.5), turned to 90 degrees
- moved D24 107.5 mm to (148.9, 104.9), turned to 180 degrees
- moved C17 107.4 mm to (151.9, 112.3), turned to 0 degrees
- moved D25 106.6 mm to (148.9, 106.4), turned to 180 degrees
- moved D26 105.7 mm to (148.9, 107.9), turned to 180 degrees
- moved U7 105.3 mm to (147.9, 106.2), turned to 0 degrees
- moved R31 105.3 mm to (145.6, 101.8), turned to 0 degrees
- moved D27 104.9 mm to (148.9, 109.4), turned to 180 degrees
- moved R32 104.3 mm to (145.6, 103.3), turned to 0 degrees
- moved D28 104.1 mm to (148.9, 111.0), turned to 180 degrees
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Connections:
- C11 pad 1: +8V -> VBAT
- C12 pad 1: +8V -> VBAT
- C2 pad 1: +8V -> VBAT
- C26 pad 1: +8V -> VBAT
- C8 pad 1: +8V -> VBAT
- D13 pad 1: +8V -> VBAT
- FAN1 pad 1: +8V -> VBAT
- Q9 pad 3: +8V -> VBAT
- R11 pad 1: +3.3V -> +5V
- R14 pad 1: +8V -> VOL_CHECK
- R14 pad 2: VOL_CHECK -> VBAT
- R15 pad 1: VOL_CHECK -> GND
- R15 pad 2: GND -> VOL_CHECK
- R3 pad 1: +3.3V -> +5V
- R5 pad 1: +3.3V -> +5V
- R8 pad 1: +3.3V -> +5V
- U2 pad 3: +8V -> VBAT
- U5 pad 13: +8V -> VBAT
- U5 pad 14: +8V -> VBAT
- U5 pad 24: +8V -> VBAT
Routing:
- net +5V: track 110.8 -> 250.8 mm, vias 0 -> 8
- net VBAT: track 0.00 -> 67.3 mm, vias 0 -> 1
- net +8V: track 59.1 -> 0.00 mm, vias 1 -> 0
- net +3.3V: track 465.8 -> 450.9 mm, vias 11 -> 13
- net GND: track 22.3 -> 14.5 mm, vias 248 -> 350
- net SENSOR_R: track 48.3 -> 55.2 mm
- net LED_6: track 52.5 -> 46.0 mm
- net MOTOR_L_OUT1: track 17.9 -> 23.7 mm
- net SD_DAT3: track 65.8 -> 60.8 mm
- net SD_DAT1: track 84.9 -> 80.5 mm, vias 6 -> 4
- net IR_FR: track 53.2 -> 57.2 mm
- net SD_DAT2: track 69.2 -> 65.4 mm
- net SENSOR_FR: track 60.7 -> 64.5 mm
- net SENSOR_L: track 50.8 -> 47.4 mm
- net SD_DAT0: track 87.5 -> 84.2 mm
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Other:
- board size 70 x 164.1 mm -> 87.3 x 100 mm
