File: yuho.kicad_sch (KiCad schematic)
At the start: 137 parts, among them J1 Conn_02x05_Odd_Even, J2 Conn_02x04_Odd_Even, J3 47219-2001, J4 Conn_02x04_Odd_Even, Q1 2N7002K, Q10 2N7002K, Q11 SSM3K344R, Q2 ST-1KL3A, Q3 2N7002K, Q4 ST-1KL3A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

Commit message: 発注用のもの(だと信じたい)ver
Parts:
- removed Q11: SSM3K344R, Fusoku:2SC2712GRLF, symbol Transistor_FET:2N7002K
- added C27: 0.1μ, Capacitor_SMD:C_0603_1608Metric_Pad1.08x0.95mm_HandSolder, symbol Device:C
- added Q12: AO3400A, Package_TO_SOT_SMD:SOT-23, symbol Transistor_FET:AO3400A
- C1: value 10μ -> 22μ; footprint Capacitor_SMD:C_0603_1608Metric_Pad1.08x0.95mm_HandSolder -> Capacitor_SMD:C_1210_3225Metric_Pad1.33x2.70mm_HandSolder
- C2: value 0.1μ -> 1.0μ
- C3: footprint Capacitor_SMD:C_0603_1608Metric_Pad1.08x0.95mm_HandSolder -> Capacitor_SMD:C_0805_2012Metric_Pad1.18x1.45mm_HandSolder
- C4: value 2.2μ -> 4.7μ; footprint Capacitor_SMD:C_0603_1608Metric_Pad1.08x0.95mm_HandSolder -> Capacitor_SMD:C_0805_2012Metric_Pad1.18x1.45mm_HandSolder
- Q9: value IRLML6402 -> AO3407A
- R11, R3, R5, R8: value 10 -> 20
- U3, U4: value ~ -> (none)
Connections:
- net +3.3V: no longer R11.1, R3.1, R5.1, R8.1
- net +5V: now also R11.1, R3.1, R5.1, R8.1
- net FAN: now also Q12.1 (G)
- net GND: now also R15.1, C27.1; no longer R15.2
- net GND2: now also Q12.2 (S)
- net VOL_CHECK: now also R14.1, R15.2, C27.2; no longer R14.2, R15.1
- net at C12.2, D13.2 (A), FAN1.2 (-): now also Q12.3 (D)
- net +8V renamed VBAT
- net VBAT: now also R14.2; no longer R14.1
Other:
- title: yuho -> yuho_ver2
- moved on the sheet: R14, R15
